File: hw/twonkie.kicad_pcb (KiCad board)
At the start: 4 copper layers, 25.4 x 25.4 mm, 60 parts, among them J1 USB4151, J2 690-024-294T331, J3 629105150521, Q1 BSD840N, Q2 BSD840N, Q3 BSD840N, Q4 BSD840N, SW1 EVQ-P7M01P, U1 INA260, U2 INA260, U3 MIC5504, U4 STM32F072CB, U5 AD8606

Commit message: wip
Parts:
- removed ?: , 
- removed DS2: CLVBA-FKA, LED_SMD:LED_Cree-PLCC4_3.2x2.8mm_CCW
- removed G***: oshw_logo_silkscreen_back_3.5mm, twonkie:oshw_logo_silkscreen_back_3.5mm
- removed R5: 620, Resistor_SMD:R_0402_1005Metric_Pad0.72x0.64mm_HandSolder
- removed R6, R7: 400, Resistor_SMD:R_0402_1005Metric_Pad0.72x0.64mm_HandSolder
- removed dojoe-logo: G***, twonkie:dojoe-logo
- C1, C3, C7, C8, C9: footprint Capacitor_SMD:C_0402_1005Metric_Pad0.74x0.62mm_HandSolder -> Capacitor_SMD:C_0402_1005Metric; moved to F.Cu
- C2, C4, C5, C6: footprint Capacitor_SMD:C_0402_1005Metric_Pad0.74x0.62mm_HandSolder -> Capacitor_SMD:C_0402_1005Metric
- D1, DS1, Q4, TP1, TP2, TP3, U1: moved to F.Cu
- FB1: footprint Inductor_SMD:L_0402_1005Metric_Pad0.77x0.64mm_HandSolder -> Inductor_SMD:L_0402_1005Metric; moved to F.Cu
- FB2: footprint Inductor_SMD:L_0402_1005Metric_Pad0.77x0.64mm_HandSolder -> Inductor_SMD:L_0402_1005Metric
- J1: footprint twonkie:GCT_USB4151_EdgeMount -> twonkie:USB_C_Plug_Wurth_632712000011
- J2: footprint twonkie:EDAC_690-024-294T331_EdgeMount -> Connector_USB:USB_C_Receptacle_Amphenol_12401548E4-2A
- J3: footprint twonkie:USB_Micro-B_Wuerth_629105150521_HandSolder -> Connector_USB:USB_Micro-B_Wuerth_629105150521
- R1, R10, R11, R12, R13, R14, R15, R16, R17, R18, R19, R20, R21, R22, R23, R24, R25, R26, R27, R8, R9: footprint Resistor_SMD:R_0402_1005Metric_Pad0.72x0.64mm_HandSolder -> Resistor_SMD:R_0402_1005Metric
- R2, R3, R4: footprint Resistor_SMD:R_0402_1005Metric_Pad0.72x0.64mm_HandSolder -> Resistor_SMD:R_0402_1005Metric; moved to F.Cu
- U3: footprint Package_TO_SOT_SMD:SOT-23-5_HandSoldering -> Package_TO_SOT_SMD:SOT-23-5; moved to F.Cu
- U4: value STM32F072CB -> STM32F072RBTx; footprint twonkie:LQFP-48_7x7mm_P0.5mm-QFN48-Frankenstein -> Package_QFP:LQFP-64_10x10mm_P0.5mm; moved to F.Cu
- moved J3 104.5 mm to (171.2, 101.0), turned to 90 degrees
- moved FB1 101.2 mm to (165.0, 103.4), turned to 90 degrees
- moved D1 100.8 mm to (166.8, 104.5), turned to -90 degrees
- moved U3 100.6 mm to (162.4, 105.8), turned to 180 degrees
- moved Q1 99.5 mm to (164.6, 88.3), turned to 90 degrees
- moved C1 99.5 mm to (165.0, 105.4), turned to -90 degrees
- moved R14 96.2 mm to (163.4, 85.8), turned to 180 degrees
- moved R15 91.2 mm to (159.9, 82.2)
- moved R13 89.3 mm to (158.9, 82.2)
- moved SW1 88.6 mm to (173.5, 91.5)
- moved R24 87.8 mm to (173.5, 95.2), turned to 180 degrees
- moved R12 87.4 mm to (157.9, 82.2)
- moved R27 87.3 mm to (170.5, 93.5), turned to -90 degrees
- moved R1 85.9 mm to (168.4, 92.5), turned to 180 degrees
- moved C8 85.6 mm to (158.5, 98.2)
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Connections:
- C5 pad 1: Net-(C5-Pad1) -> /VDDA
- C6 pad 1: Net-(C5-Pad1) -> /VDDA
- FB2 pad 2: Net-(C5-Pad1) -> /VDDA
- U1 pad 13: Net-(U1-Pad13) -> unconnected-(U1-Pad13)
- U3 pad 4: Net-(U3-Pad4) -> unconnected-(U3-Pad4)
- U4 pad 10: /CC1_EN -> /CC2_RPUSB
- U4 pad 11: /CC1_BUF -> /CC2_RD
- U4 pad 12: /CC2_EN -> GND
- U4 pad 13: /CC2_BUF -> /VDDA
- U4 pad 14: /DAC -> /CC2_RA
- U4 pad 15: /TX_CLK -> /CC2_RP1A5
- U4 pad 16: /CC2_TX_DATA -> /CC2_RP3A0
- U4 pad 17: /VCONN_ALERT_L -> /CC1_BUF
- U4 pad 18: Net-(U4-Pad18) -> GND
- U4 pad 19: Net-(U4-Pad19) -> +3V3
- U4 pad 2: /CC2_TX_EN -> /CC1_RPUSB
- U4 pad 20: /VBUS_ALERT_L -> /CC2_BUF
- U4 pad 21: /LED_G_L -> /TX_CLK
- U4 pad 22: /LED_R_L -> /CC2_TX_DATA
- U4 pad 23: GND -> /CC2_TX_EN
- U4 pad 24: +3V3 -> unconnected-(U4-Pad24)
- U4 pad 25: /CC2_RPUSB -> unconnected-(U4-Pad25)
- U4 pad 26: /CC2_RD -> unconnected-(U4-Pad26)
- U4 pad 27: /LED_B_L -> /VCONN_ALERT_L
- U4 pad 28: /CC2_RP1A5 -> /VBUS_ALERT_L
- U4 pad 29: /CC2_RA -> /INA_SCL
- U4 pad 3: /CC1_RP3A0 -> /CC1_RD
- U4 pad 30: /UART_TX -> /INA_SDA
- U4 pad 31: /UART_RX -> GND
- U4 pad 32: /USB_B_D- -> +3V3
- U4 pad 33: /USB_B_D+ -> unconnected-(U4-Pad33)
- U4 pad 34: /CC2_RP3A0 -> unconnected-(U4-Pad34)
- U4 pad 35: GND -> unconnected-(U4-Pad35)
- U4 pad 36: +3V3 -> unconnected-(U4-Pad36)
- U4 pad 37: /CC1_TX_EN -> unconnected-(U4-Pad37)
- U4 pad 38: /CC1_RPUSB -> unconnected-(U4-Pad38)
- U4 pad 39: /CC1_RD -> unconnected-(U4-Pad39)
- U4 pad 4: Net-(U4-Pad4) -> /CC1_RA
- U4 pad 40: /CC1_TX_DATA -> unconnected-(U4-Pad40)
- U4 pad 41: /CC1_RP1A5 -> unconnected-(U4-Pad41)
- U4 pad 42: /INA_SCL -> /UART_TX
- U4 pad 43: /INA_SDA -> /UART_RX
- U4 pad 44: /BOOT -> /USB_B_D-
- U4 pad 45: /CC1_RA -> /USB_B_D+
- U4 pad 46: /TX_CLK -> /SWDIO
- U4 pad 5: /OSC_IN -> /CC1_RP1A5
- U4 pad 6: /OSC_OUT -> /CC1_RP3A0
- U4 pad 8: GND -> /CC1_EN
- U4 pad 9: Net-(C5-Pad1) -> /CC2_EN
Routing:
- net GND: track 64.0 -> 22.5 mm, vias 31 -> 0
- net +3V3: track 45.6 -> 4.13 mm, vias 12 -> 0
- net /CC1: track 18.3 -> 46.0 mm, vias 0 -> 4
- net /CC1_RECEP: track 23.8 -> 0.00 mm, vias 4 -> 0
- net /CC2_RECEP: track 9.94 -> 30.4 mm, vias 2 -> 0
- net /TX2-: track 19.0 -> 0.00 mm
- net /TX2+: track 19.0 -> 0.00 mm
- net /USBC_D+: track 18.4 -> 0.00 mm, vias 1 -> 0
- net /TX1-: track 18.3 -> 0.00 mm
- net /TX1+: track 18.3 -> 0.00 mm
- net /RX1-: track 18.3 -> 0.00 mm
- net /RX1+: track 18.3 -> 0.00 mm
- net /USBC_D-: track 17.2 -> 0.00 mm, vias 1 -> 0
- net /SBU2: track 17.2 -> 0.00 mm, vias 2 -> 0
- net /SBU1: track 16.5 -> 0.00 mm, vias 2 -> 0
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- removed copper zone on B.Cu, net +3V3
- removed copper zone on In1.Cu, net +3V3
- removed copper zone on In2.Cu, net +3V3
- removed copper zone on B.Cu, net +5V
- removed copper zone on B.Cu, net /CC2_PLUG
- removed copper zone on F.Cu, net /CC2_PLUG
- removed copper zone on B.Cu, net /CC2_RECEP
- removed copper zone on F.Cu, net /CC2_RECEP
- removed copper zone on B.Cu, net /VBUS_PLUG
- removed copper zone on F.Cu, net /VBUS_PLUG
- removed copper zone on In2.Cu, net /VBUS_PLUG
- removed copper zone on B.Cu, net /VBUS_RECEP
- removed copper zone on F.Cu, net /VBUS_RECEP
- removed copper zone on In2.Cu, net /VBUS_RECEP
- removed copper zone on B.Cu, net GND
- removed copper zone on F.Cu, net GND
- removed copper zone on In1.Cu, net GND
- removed copper zone on In2.Cu, net GND
Other:
- board size 25.4 x 25.4 mm -> 50 x 50 mm
- net class Default removed
- net class Diffpair removed
- net class Power removed
- board text removed: "2020"
- board text removed: "Based on Google's Twinkie"
- board text removed: "Twonkie USB PD Sniffer"
- board text removed: "v1.0"
